File: pcb/ESPLeveller/ESPLeveller.kicad_pcb (KiCad board)
At the start: 2 copper layers, 105 x 75 mm, 12 parts, among them J1 Battery_18650x2, J2 Sensor_Pod, J3 OPT_BTN, SW1 PWR, U1 ESP32C3_SuperMini, U2 TP4056_ChargeProt, U3 MT3608_5V

Commit message: feat(pcb): P2.5 — placement re-optimization + 3D component models
Layout iteration driven by real-module dimensions and the design
checklist:
- SuperMini antenna section now overhangs the east board edge
  (RF rule: no copper under antenna) with an explicit rule-area
  keepout blocking tracks/vias/pads/pour in the overhang zone
- TP4056 USB end overhangs west edge (charge cable access)
- SW1 actuator faces the top board edge (finger-accessible; was
  default-rotated inward — user catch)
- real-body collision pass found 3 clashes invisible to courtyard
  DRC (module bodies wider than courtyards): J1/C1/D1/J3 moved
- all 12 components have 3D models (stock STEP + simple WRL boxes
  for the module footprints) so the assembled render shows the
  actual build
DRC: 0 errors, 0 unconnected (5 silk warnings). ERC: 0 errors.
Parts:
- moved U1 14.0 mm to (114.0, 55.0)
- moved J1 6.00 mm to (35.0, 76.0)
- moved C1 4.00 mm to (66.0, 74.0)
- moved J3 4.00 mm to (95.0, 86.0)
- moved D1 2.00 mm to (95.0, 76.0)
- moved SW1 2.00 mm to (49.0, 60.0), turned to 90 degrees
Routing:
- net GND: track 155.0 -> 0.00 mm
- net +5V: track 39.6 -> 57.6 mm
- net /LED_STAT: track 14.2 -> 28.2 mm
- net +3V3: track 41.3 -> 55.3 mm
- net /BTN: track 20.2 -> 28.6 mm
- net Net-(U3-IN+): track 6.69 -> 15.1 mm
- net /BATT-: track 15.1 -> 21.1 mm
- net /BATT+: track 12.6 -> 18.6 mm
- net /SDA: track 33.4 -> 39.0 mm
- net /SCL: track 49.6 -> 45.9 mm
- net Net-(U2-OUT+): track 18.3 -> 16.3 mm
- net Net-(D1-Pad2): track 5.53 -> 3.53 mm
